Commit message: [ADDED & UPDATED] the robot to spawn with the UR5e at a home position, had to change some parameters in the xacro, and install some files for ros2_control

File: components/common_macro/mpo_cabinet_macro.xacro (robot description, xacro)
@@ -32,5 +32,5 @@
                 <origin rpy="${collision_rpy}" xyz="0 0 0"/>
                 <geometry>
-                    <mesh filename="package://steve_simulation/robots/${neo_robot_name}/meshes/cabin.dae" scale="${model_scale}"/>
+                    <mesh filename="package://steve_simulation/robots/${neo_robot_name}/meshes/cabin.stl" scale="${model_scale}"/>
                 </geometry>
             </collision>

File: robots/mmo_700/urdf/macro/mpo_700_caster.xacro (robot description, xacro)
@@ -1,9 +1,8 @@
 <?xml version="1.0"?>
 <robot xmlns:xacro="http://www.ros.org/wiki/xacro" name="mpo_700">
-  <xacro:macro name="mpo_700_caster_0" params="name parent *origin">
+  <xacro:macro name="mpo_700_caster_body" params="name parent *origin">
    <joint name="${name}_joint" type="fixed">
     <xacro:insert_block name="origin" />
     <axis xyz="0 0 -1" />
-    <!-- <limit effort="1000.0" lower="-1e+16" upper="1e+16" velocity="3.5"/> -->
     <joint_properties damping="1" friction="1" />
     <parent link="${parent}" />
@@ -13,6 +12,6 @@
     <inertial>
       <mass value="9" />
-      <origin xyz="0 0 0" rpy="0 0 0" />
-      <inertia ixx="0.00044332" ixy="0" ixz="0" iyy="0.00044332" iyz="0" izz="0.00072" />
+      <origin xyz="0 0 0.05" rpy="0 0 0" />
+      <inertia ixx="0.04" ixy="0" ixz="0" iyy="0.04" iyz="0" izz="0.04" />
     </inertial>
     <visual>
@@ -25,92 +24,28 @@
      <origin xyz="0 0 0.10" rpy="0 0 0" />
      <geometry>
-        <mesh filename="package://steve_simulation/robots/mmo_700/meshes/MPO-700-HEAD.dae" scale="0.001 0.001 0.001"/>
+        <mesh filename="package://steve_simulation/robots/mmo_700/meshes/MPO-700-HEAD.stl" scale="0.001 0.001 0.001"/>
      </geometry>
     </collision>
    </link>
   </xacro:macro>
+  <xacro:macro name="mpo_700_caster_0" params="name parent *origin">
+    <xacro:mpo_700_caster_body name="${name}" parent="${parent}">
+      <xacro:insert_block name="origin"/>
+    </xacro:mpo_700_caster_body>
+  </xacro:macro>
   <xacro:macro name="mpo_700_caster_1" params="name parent *origin">
-   <joint name="${name}_joint" type="fixed">
-    <xacro:insert_block name="origin" />
-    <axis xyz="0 0 -1" />
-    <joint_properties damping="1" friction="1" />
-    <parent link="${parent}" />
-    <child link="${name}_link" />
-   </joint>
-   <link name="${name}_link">
-    <inertial>
-      <mass value="9" />
-      <origin xyz="0 0 0." rpy="0 0 0" />
-      <inertia ixx="0.00044332" ixy="0" ixz="0" iyy="0.00044332" iyz="0" izz="0.00072" />
-    </inertial>
-    <visual>
-     <origin xyz="0 0 0.10" rpy="0 0 0"/>
-     <geometry>
-        <mesh filename="package://steve_simulation/robots/mmo_700/meshes/MPO-700-HEAD.dae" scale="0.001 0.001 0.001"/>
-     </geometry>
-    </visual>
-    <collision>
-     <origin xyz="0 0 0.10" rpy="0 0 0" />
-     <geometry>
-        <mesh filename="package://steve_simulation/robots/mmo_700/meshes/MPO-700-HEAD.dae" scale="0.001 0.001 0.001"/>
-     </geometry>
-    </collision>
-   </link>
+    <xacro:mpo_700_caster_body name="${name}" parent="${parent}">
+      <xacro:insert_block name="origin"/>
+    </xacro:mpo_700_caster_body>
   </xacro:macro>
   <xacro:macro name="mpo_700_caster_2" params="name parent *origin">
-   <joint name="${name}_joint" type="fixed">
-    <xacro:insert_block name="origin" />
-    <axis xyz="0 0 -1" />
-    <joint_properties damping="1" friction="1" />
-    <parent link="${parent}" />
-    <child link="${name}_link" />
-   </joint>
-   <link name="${name}_link">
-    <inertial>
-      <mass value="9" />
-      <origin xyz="0 0 0." rpy="0 0 0" />
-      <inertia ixx="0.00044332" ixy="0" ixz="0" iyy="0.00044332" iyz="0" izz="0.00072" />
-    </inertial>
-    <visual>
-     <origin xyz="0 0 0.10" rpy="0 0 0"/>
-     <geometry>
-        <mesh filename="package://steve_simulation/robots/mmo_700/meshes/MPO-700-HEAD.dae" scale="0.001 0.001 0.001"/>
-     </geometry>
-    </visual>
-    <collision>
-     <origin xyz="0 0 0.10" rpy="0 0 0" />
-     <geometry>
-        <mesh filename="package://steve_simulation/robots/mmo_700/meshes/MPO-700-HEAD.dae" scale="0.001 0.001 0.001"/>
-     </geometry>
-    </collision>
-   </link>
+    <xacro:mpo_700_caster_body name="${name}" parent="${parent}">
+      <xacro:insert_block name="origin"/>
+    </xacro:mpo_700_caster_body>
   </xacro:macro>
   <xacro:macro name="mpo_700_caster_3" params="name parent *origin">
-   <joint name="${name}_joint" type="fixed">
-    <xacro:insert_block name="origin" />
-    <axis xyz="0 0 -1" />
-    <joint_properties damping="1" friction="1" />
-    <parent link="${parent}" />
-    <child link="${name}_link" />
-   </joint>
-   <link name="${name}_link">
-    <inertial>
-      <mass value="9" />
-      <origin xyz="0 0 0" rpy="0 0 0" />
-      <inertia ixx="0.00044332" ixy="0" ixz="0" iyy="0.00044332" iyz="0" izz="0.00072" />
-    </inertial>
-    <visual>
-     <origin xyz="0 0 0.10" rpy="0 0 0"/>
-     <geometry>
-        <mesh filename="package://steve_simulation/robots/mmo_700/meshes/MPO-700-HEAD.dae" scale="0.001 0.001 0.001"/>
-     </geometry>
-    </visual>
-    <collision>
-     <origin xyz="0 0 0.10" rpy="0 0 0" />
-     <geometry>
-        <mesh filename="package://steve_simulation/robots/mmo_700/meshes/MPO-700-HEAD.dae" scale="0.001 0.001 0.001"/>
-     </geometry>
-    </collision>
-   </link>
+    <xacro:mpo_700_caster_body name="${name}" parent="${parent}">
+      <xacro:insert_block name="origin"/>
+    </xacro:mpo_700_caster_body>
   </xacro:macro>
 </robot>

File: robots/mmo_700/urdf/macro/mpo_700_wheel.xacro (robot description, xacro)
@@ -26,14 +26,8 @@
      <origin xyz="0 0 0" rpy="0 0 0" />
      <geometry>
-        <mesh filename="package://steve_simulation/robots/mmo_700/meshes/MPO-700-WHEEL.dae" scale="0.001 0.001 0.001"/>
+        <mesh filename="package://steve_simulation/robots/mmo_700/meshes/MPO-700-WHEEL.stl" scale="0.001 0.001 0.001"/>
      </geometry>
     </collision>
    </link>
-     <gazebo reference="${name}_link">
-      <mu1 value="0.05"/>
-      <mu2 value="0.05"/>
-      <kp value="100000.0" />
-      <kd value="10.0" />
-      </gazebo>
   </xacro:macro>
 </robot>

File: robots/mmo_700/urdf/mmo_700_body.urdf.xacro (robot description, xacro)
@@ -15,7 +15,7 @@
         </visual>
         <collision>
-            <origin rpy="0 0 -1.571" xyz="0. 0. 0."/>
+            <origin rpy="0 0 -1.571" xyz="0.0 0.0 0.0"/>
             <geometry>
-                <mesh filename="package://steve_simulation/robots/mmo_700/meshes/MPO-700-BODY.dae" scale="0.001 0.001 0.001"/>
+                <mesh filename="package://steve_simulation/robots/mmo_700/meshes/MPO-700-BODY.stl" scale="0.001 0.001 0.001"/>
             </geometry>
         </collision>

File: robots/mmo_700/urdf/mmo_700_gazebo.urdf.xacro (robot description, xacro)
@@ -47,28 +47,26 @@
         visualize="false"
     />
-    <!--Wheels - Gazebo friction properties-->
-    <gazebo reference="mpo_700_wheel_front_left_link">
-      <mu1>0.05</mu1>
-      <mu2>0.05</mu2>
-      <kp>100000.0</kp>
-      <kd>10.0</kd>
-    </gazebo>
-    <gazebo reference="mpo_700_wheel_front_right_link">
-      <mu1>0.05</mu1>
-      <mu2>0.05</mu2>
-      <kp>100000.0</kp>
-      <kd>10.0</kd>
-    </gazebo>
-    <gazebo reference="mpo_700_wheel_back_left_link">
-      <mu1>0.05</mu1>
-      <mu2>0.05</mu2>
-      <kp>100000.0</kp>
-      <kd>10.0</kd>
-    </gazebo>
-    <gazebo reference="mpo_700_wheel_back_right_link">
-      <mu1>0.05</mu1>
-      <mu2>0.05</mu2>
-      <kp>100000.0</kp>
-      <kd>10.0</kd>
-    </gazebo>
+    <!-- Enough friction to hold station against mesh-contact drift, but well
+         below the mu that made teleop tip the base. slip lets planar_move slide. -->
+    <xacro:macro name="mpo_700_ground_contact" params="link">
+      <gazebo reference="${link}">
+        <mu1>0.2</mu1>
+        <mu2>0.2</mu2>
+        <slip1>0.2</slip1>
+        <slip2>0.2</slip2>
+        <kp>1e7</kp>
+        <kd>1e2</kd>
+        <minDepth>0.001</minDepth>
+        <maxVel>0.1</maxVel>
+      </gazebo>
+    </xacro:macro>
+    <xacro:mpo_700_ground_contact link="base_link"/>
+    <xacro:mpo_700_ground_contact link="mpo_700_wheel_front_left_link"/>
+    <xacro:mpo_700_ground_contact link="mpo_700_wheel_front_right_link"/>
+    <xacro:mpo_700_ground_contact link="mpo_700_wheel_back_left_link"/>
+    <xacro:mpo_700_ground_contact link="mpo_700_wheel_back_right_link"/>
+    <xacro:mpo_700_ground_contact link="mpo_700_caster_front_left_link"/>
+    <xacro:mpo_700_ground_contact link="mpo_700_caster_front_right_link"/>
+    <xacro:mpo_700_ground_contact link="mpo_700_caster_back_left_link"/>
+    <xacro:mpo_700_ground_contact link="mpo_700_caster_back_right_link"/>
 </robot>
