Commit message: " [UPDATED]  with the robotiq wrist and the navigation and simulation readme "

File: src/steve_simulation/components/arm/ur_arm.urdf.xacro (robot description, xacro)
@@ -19,4 +19,7 @@
             <xacro:arg name="simulation_controllers" default="$(find steve_simulation)/configs/ur_config/$(arg arm_type)/ur_controllers.yaml"/>
             <xacro:arg name="initial_positions_file" default="$(find steve_simulation)/configs/ur_config/initial_joint_positions.yaml"/>
+            <xacro:arg name="arm_tool" default="robotiq_gripper"/>
+            <xacro:arg name="include_wrist_camera" default="true"/>
+            <xacro:property name="arm_tool" value="$(arg arm_tool)"/>
             <!-- parse initial positions as a dictionary -->
             <xacro:property
@@ -54,5 +57,11 @@
                 </gazebo>
             </xacro:if>
-            <!-- include wrist camera mount (dummy end-effector with camera) -->
-            <xacro:include filename="$(find steve_simulation)/components/arm/wrist_camera_mount.urdf.xacro"/>
+            <!-- Robotiq 2F-85 gripper on the UR tool flange -->
+            <xacro:if value="${arm_tool == 'robotiq_gripper'}">
+                <xacro:include filename="$(find steve_simulation)/components/arm/robotiq_gripper.urdf.xacro"/>
+            </xacro:if>
+            <!-- Wrist D405 camera, mounted on tool0 (with or without gripper) -->
+            <xacro:if value="$(arg include_wrist_camera)">
+                <xacro:include filename="$(find steve_simulation)/components/arm/wrist_camera_mount.urdf.xacro"/>
+            </xacro:if>
 </robot>

File: src/steve_simulation/components/arm/wrist_camera_mount.urdf.xacro (robot description, xacro)
@@ -1,41 +1,9 @@
 <?xml version="1.0"?>
-<!-- Dummy end-effector with wrist camera for real robot (no gripper) -->
+<!-- Wrist D405 camera mounted on the UR tool flange. -->
 <robot xmlns:xacro="http://www.ros.org/wiki/xacro" name="wrist_camera_mount">
-            <!-- Get tf_prefix from parent scope -->
             <xacro:arg name="tf_prefix" default="ur5e"/>
             <xacro:property name="tf_prefix" value="$(arg tf_prefix)"/>
             <xacro:arg name="use_gazebo" default="true"/>
-            <material name="mount_grey">
-              <color rgba="0.7 0.7 0.7 1"/>
-            </material>
-            <!-- Dummy end-effector link (replaces gripper adapter) -->
-            <joint name="tool0_to_dummy_ee_joint" type="fixed">
-              <parent link="${tf_prefix}tool0"/>
-              <child link="dummy_end_effector"/>
-              <origin xyz="0 0 0" rpy="0 0 0"/>
-            </joint>
-            <link name="dummy_end_effector">
-              <visual>
-                <origin xyz="0 0 0.025" rpy="0 0 0"/>
-                <geometry>
-                  <!-- Simple cylinder representing the mounting plate -->
-                  <cylinder radius="0.04" length="0.05"/>
-                </geometry>
-                <material name="mount_grey"/>
-              </visual>
-              <collision>
-                <origin xyz="0 0 0.025" rpy="0 0 0"/>
-                <geometry>
-                  <cylinder radius="0.04" length="0.05"/>
-                </geometry>
-              </collision>
-              <inertial>
-                <mass value="0.2"/>
-                <origin xyz="0 0 0.025" rpy="0 0 0"/>
-                <inertia ixx="0.0001" ixy="0" ixz="0" iyy="0.0001" iyz="0" izz="0.0001"/>
-              </inertial>
-            </link>
-            <!-- Include wrist camera -->
             <xacro:include filename="$(find steve_simulation)/components/cameras/wrist_d405.urdf.xacro"/>
-            <xacro:wrist_d405 parent="dummy_end_effector" use_gazebo="$(arg use_gazebo)"/>
+            <xacro:wrist_d405 parent="${tf_prefix}tool0" use_gazebo="$(arg use_gazebo)"/>
 </robot>
