Commit message: [UPDATED] for the manipulation stack and pick up sequence

File: src/steve_simulation/components/arm/robotiq_gripper.urdf.xacro (robot description, xacro)
@@ -12,9 +12,7 @@
       rotation="${pi/2}"
       />
-  <!-- 2F-85 kinematics and meshes. ros2_control is omitted because the
-       upstream sim_gazebo flag targets gz_ros2_control (Ignition), not
-       Gazebo Classic used by this workspace. Finger joints are still in
-       the URDF as revolute/mimic; simulation.launch.py fills them in for
-       robot_state_publisher so RViz can show the fingers. -->
+  <!-- 2F-85 kinematics and meshes. Upstream ros2_control is omitted because
+       its sim_gazebo flag loads gz_ros2_control (Ignition). Classic Gazebo
+       hardware is added below as gazebo_ros2_control/GazeboSystem. -->
   <xacro:include filename="$(find robotiq_description)/urdf/robotiq_2f_85_macro.urdf.xacro"/>
   <xacro:robotiq_gripper
@@ -25,5 +23,61 @@
     <origin xyz="0 0 0" rpy="0 0 -${pi / 2}"/>
   </xacro:robotiq_gripper>
-  <!-- Gazebo Classic appearance and keep the fingers from sagging. -->
+  <!-- Grasp frame used as the MoveIt tip. 0.148 m is about the 2F-85 palm-to-pad distance. -->
+  <link name="gripper_tcp"/>
+  <joint name="gripper_tcp_joint" type="fixed">
+    <parent link="robotiq_85_base_link"/>
+    <child link="gripper_tcp"/>
+    <origin xyz="0 0 0.148" rpy="0 0 0"/>
+  </joint>
+  <!-- Gazebo Classic hardware. robotiq_description's sim_gazebo flag loads
+       gz_ros2_control (Ignition), which this workspace does not use. -->
+  <ros2_control name="robotiq_gripper" type="system">
+    <hardware>
+      <plugin>gazebo_ros2_control/GazeboSystem</plugin>
+    </hardware>
+    <joint name="robotiq_85_left_knuckle_joint">
+      <command_interface name="position"/>
+      <state_interface name="position">
+        <param name="initial_value">0.0</param>
+      </state_interface>
+      <state_interface name="velocity"/>
+    </joint>
+    <joint name="robotiq_85_right_knuckle_joint">
+      <param name="mimic">robotiq_85_left_knuckle_joint</param>
+      <param name="multiplier">-1</param>
+      <command_interface name="position"/>
+      <state_interface name="position"/>
+      <state_interface name="velocity"/>
+    </joint>
+    <joint name="robotiq_85_left_inner_knuckle_joint">
+      <param name="mimic">robotiq_85_left_knuckle_joint</param>
+      <param name="multiplier">1</param>
+      <command_interface name="position"/>
+      <state_interface name="position"/>
+      <state_interface name="velocity"/>
+    </joint>
+    <joint name="robotiq_85_right_inner_knuckle_joint">
+      <param name="mimic">robotiq_85_left_knuckle_joint</param>
+      <param name="multiplier">-1</param>
+      <command_interface name="position"/>
+      <state_interface name="position"/>
+      <state_interface name="velocity"/>
+    </joint>
+    <joint name="robotiq_85_left_finger_tip_joint">
+      <param name="mimic">robotiq_85_left_knuckle_joint</param>
+      <param name="multiplier">-1</param>
+      <command_interface name="position"/>
+      <state_interface name="position"/>
+      <state_interface name="velocity"/>
+    </joint>
+    <joint name="robotiq_85_right_finger_tip_joint">
+      <param name="mimic">robotiq_85_left_knuckle_joint</param>
+      <param name="multiplier">1</param>
+      <command_interface name="position"/>
+      <state_interface name="position"/>
+      <state_interface name="velocity"/>
+    </joint>
+  </ros2_control>
+  <!-- Gazebo Classic appearance. Gravity is off so idle fingers do not sag. -->
   <xacro:if value="$(arg use_gazebo)">
     <xacro:macro name="robotiq_gazebo_link" params="link">
@@ -43,18 +97,4 @@
     <xacro:robotiq_gazebo_link link="robotiq_85_left_finger_tip_link"/>
     <xacro:robotiq_gazebo_link link="robotiq_85_right_finger_tip_link"/>
-    <xacro:macro name="robotiq_hold_joint" params="joint">
-      <gazebo reference="${joint}">
-        <implicitSpringDamper>true</implicitSpringDamper>
-        <springStiffness>10000</springStiffness>
-        <springReference>0.0</springReference>
-        <dissipation>1.0</dissipation>
-      </gazebo>
-    </xacro:macro>
-    <xacro:robotiq_hold_joint joint="robotiq_85_left_knuckle_joint"/>
-    <xacro:robotiq_hold_joint joint="robotiq_85_right_knuckle_joint"/>
-    <xacro:robotiq_hold_joint joint="robotiq_85_left_inner_knuckle_joint"/>
-    <xacro:robotiq_hold_joint joint="robotiq_85_right_inner_knuckle_joint"/>
-    <xacro:robotiq_hold_joint joint="robotiq_85_left_finger_tip_joint"/>
-    <xacro:robotiq_hold_joint joint="robotiq_85_right_finger_tip_joint"/>
   </xacro:if>
 </robot>

File: src/steve_simulation/components/dynamixel/steve_pan_tilt.xacro (robot description, xacro)
@@ -4,5 +4,5 @@
   <xacro:include filename="$(find steve_simulation)/components/dynamixel/dynamixel_bracket_fr12_h101.urdf.xacro" />
   <xacro:arg name="grasp_link_offset" default="0.11"/>
-+  <xacro:macro name="steve_pan_tilt" params="parent name">
+  <xacro:macro name="steve_pan_tilt" params="parent name">
     <!-- Pan motor -->
     <xacro:dynamixel_motor_XL-430 name="${name}_tilt_motor" parent="${parent}" motor_direction="-1" position_offset="0.065">

Commit message: [UPDATED] with gripper configuration, no collision, no tipping of the robot due to extension of the arm

File: src/steve_simulation/components/arm/robotiq_gripper.urdf.xacro (robot description, xacro)
@@ -31,5 +31,12 @@
   </joint>
   <!-- Gazebo Classic hardware. robotiq_description's sim_gazebo flag loads
-       gz_ros2_control (Ignition), which this workspace does not use. -->
+       gz_ros2_control (Ignition), which this workspace does not use.
+       gazebo_ros2_control 0.4 does not read URDF <mimic> tags. Each follower
+       has to be listed here with a mimic param, or the right finger, inner
+       knuckles, and finger tips stay free revolute joints in Gazebo.
+       The gripper controller still commands only the left knuckle. This
+       plugin copies that position onto the followers (with the multiplier)
+       and exports their command interfaces as *_mimic so nothing else
+       claims them. -->
   <ros2_control name="robotiq_gripper" type="system">
     <hardware>

File: src/steve_simulation/components/arm/ur_arm.urdf.xacro (robot description, xacro)
@@ -22,4 +22,10 @@
             <xacro:arg name="include_wrist_camera" default="true"/>
             <xacro:property name="arm_tool" value="$(arg arm_tool)"/>
+            <!-- Catalog UR5e mass pitches the base when the arm stretches out.
+                 Use the 1/5 mass and inertia file for that arm. -->
+            <xacro:property name="ur_arm_type" value="$(arg arm_type)"/>
+            <xacro:property name="stock_physical_params" value="$(arg physical_params)"/>
+            <xacro:property name="light_ur5e_physical_params" value="$(find steve_simulation)/configs/ur_config/ur5e/physical_parameters.yaml"/>
+            <xacro:property name="resolved_physical_params" value="${light_ur5e_physical_params if ur_arm_type == 'ur5e' else stock_physical_params}"/>
             <!-- parse initial positions as a dictionary -->
             <xacro:property
@@ -33,5 +39,5 @@
                 joint_limits_parameters_file="$(arg joint_limit_params)"
                 kinematics_parameters_file="$(arg kinematics_params)"
-                physical_parameters_file="$(arg physical_params)"
+                physical_parameters_file="${resolved_physical_params}"
                 visual_parameters_file="$(arg visual_params)"
                 safety_limits="$(arg safety_limits)"

File: src/steve_simulation/components/common_macro/gazebo_object_controller_macro.xacro (robot description, xacro)
@@ -17,5 +17,5 @@
                 <!-- Set odom publish rate -->
                 <odometryRate>${odom_update_rate}</odometryRate>
-                <!-- Set control loop update rate -->
+                <update_rate>${controller_update_rate}</update_rate>
                 <publish_rate>${controller_update_rate}</publish_rate>
                 <!-- Set if odom required -->
