Commit message: Store simulation PNG textures in Git LFS

File: src/steve_simulation/robots/mmo_700/urdf/macro/mpo_700_wheel.xacro (robot description, xacro)
@@ -24,7 +24,7 @@
     </visual>
     <collision>
-     <origin xyz="0 0 0" rpy="0 0 0" />
+     <origin xyz="0 0 0" rpy="0 1.5707963 0" />
      <geometry>
-        <mesh filename="package://steve_simulation/robots/mmo_700/meshes/MPO-700-WHEEL.stl" scale="0.001 0.001 0.001"/>
+        <cylinder radius="0.09" length="0.03"/>
      </geometry>
     </collision>

File: src/steve_simulation/robots/mmo_700/urdf/mmo_700_body.urdf.xacro (robot description, xacro)
@@ -4,7 +4,9 @@
     <link name="base_link">
         <inertial>
-            <mass value="200"/>
-            <origin xyz="0 0 0"/>
-            <inertia ixx="7.8" ixy="0.0" ixz="0" iyy="7.8" iyz="0.0" izz="7.8"/>
+            <mass value="240"/>
+            <origin xyz="0 0 0.08"/>
+            <inertia ixx="6.002" ixy="0.0" ixz="0.0"
+                     iyy="8.738" iyz="0.0"
+                     izz="13.140"/>
         </inertial>
         <visual>

File: src/steve_simulation/robots/mmo_700/urdf/mmo_700_gazebo.urdf.xacro (robot description, xacro)
@@ -47,26 +47,27 @@
         visualize="false"
     />
-    <!-- Enough friction to hold station against mesh-contact drift, but well
-         below the mu that made teleop tip the base. slip lets planar_move slide. -->
-    <xacro:macro name="mpo_700_ground_contact" params="link">
+    <xacro:macro name="mpo_700_wheel_contact" params="link">
       <gazebo reference="${link}">
-        <mu1>0.2</mu1>
-        <mu2>0.2</mu2>
-        <slip1>0.2</slip1>
-        <slip2>0.2</slip2>
-        <kp>1e7</kp>
-        <kd>1e2</kd>
+        <mu1>0.15</mu1>
+        <mu2>0.15</mu2>
+        <slip1>0.1</slip1>
+        <slip2>0.1</slip2>
+        <kp>2e5</kp>
+        <kd>80</kd>
         <minDepth>0.001</minDepth>
         <maxVel>0.1</maxVel>
       </gazebo>
     </xacro:macro>
-    <xacro:mpo_700_ground_contact link="base_link"/>
-    <xacro:mpo_700_ground_contact link="mpo_700_wheel_front_left_link"/>
-    <xacro:mpo_700_ground_contact link="mpo_700_wheel_front_right_link"/>
-    <xacro:mpo_700_ground_contact link="mpo_700_wheel_back_left_link"/>
-    <xacro:mpo_700_ground_contact link="mpo_700_wheel_back_right_link"/>
-    <xacro:mpo_700_ground_contact link="mpo_700_caster_front_left_link"/>
-    <xacro:mpo_700_ground_contact link="mpo_700_caster_front_right_link"/>
-    <xacro:mpo_700_ground_contact link="mpo_700_caster_back_left_link"/>
-    <xacro:mpo_700_ground_contact link="mpo_700_caster_back_right_link"/>
+    <xacro:mpo_700_wheel_contact link="mpo_700_wheel_front_left_link"/>
+    <xacro:mpo_700_wheel_contact link="mpo_700_wheel_front_right_link"/>
+    <xacro:mpo_700_wheel_contact link="mpo_700_wheel_back_left_link"/>
+    <xacro:mpo_700_wheel_contact link="mpo_700_wheel_back_right_link"/>
+    <gazebo reference="base_link">
+      <mu1>0.0</mu1>
+      <mu2>0.0</mu2>
+      <kp>1e4</kp>
+      <kd>10.0</kd>
+      <minDepth>0.001</minDepth>
+      <maxVel>0.1</maxVel>
+    </gazebo>
 </robot>
