Commit message: [UPDATED] with the pan tilt angle, made changes to the config file of the base, changes in inital position of the arm pose, and then added the geomentry_msgs

File: src/steve_simulation/components/cameras/l515_simplified.urdf.xacro (robot description, xacro)
@@ -54,6 +54,6 @@
             <horizontal_fov>${70*pi/180}</horizontal_fov>
             <image>
-              <width>640</width>
-              <height>480</height>
+              <width>1280</width>
+              <height>960</height>
               <format>R8G8B8</format>
             </image>
@@ -65,10 +65,13 @@
           <plugin name="${name}_controller" filename="libgazebo_ros_camera.so">
             <ros>
+              <!-- The plugin advertises ${name}/image_raw inside this
+                   namespace, so the published name is /${name}/${name}/image_raw
+                   unless this remap matches that full relative name. -->
               <namespace>${name}</namespace>
-              <remapping>image_raw:=color/image_raw</remapping>
-              <remapping>camera_info:=color/camera_info</remapping>
-              <remapping>depth/image_raw:=aligned_depth_to_color/image_raw</remapping>
-              <remapping>depth/camera_info:=aligned_depth_to_color/camera_info</remapping>
-              <remapping>points:=depth/color/points</remapping>
+              <remapping>${name}/image_raw:=color/image_raw</remapping>
+              <remapping>${name}/camera_info:=color/camera_info</remapping>
+              <remapping>${name}/depth/image_raw:=aligned_depth_to_color/image_raw</remapping>
+              <remapping>${name}/depth/camera_info:=aligned_depth_to_color/camera_info</remapping>
+              <remapping>${name}/points:=depth/color/points</remapping>
             </ros>
             <camera_name>${name}</camera_name>

File: src/steve_simulation/components/cameras/wrist_d405.urdf.xacro (robot description, xacro)
@@ -91,6 +91,7 @@
         <horizontal_fov>${80.4*pi/180}</horizontal_fov>
         <image>
-          <width>640</width>
-          <height>480</height>
+          <!-- 1280 keeps a 40 mm cube above ~15 px at the 1.5 m spawn standoff. -->
+          <width>1280</width>
+          <height>960</height>
           <format>R8G8B8</format>
         </image>
@@ -102,10 +103,13 @@
       <plugin name="wrist_camera_controller" filename="libgazebo_ros_camera.so">
         <ros>
+          <!-- The plugin advertises wrist_camera/image_raw inside this
+               namespace. Remapping the bare name image_raw does not match,
+               and the picture never reaches color/image_raw. -->
           <namespace>wrist_camera</namespace>
-          <remapping>image_raw:=color/image_raw</remapping>
-          <remapping>camera_info:=color/camera_info</remapping>
-          <remapping>depth/image_raw:=aligned_depth_to_color/image_raw</remapping>
-          <remapping>depth/camera_info:=aligned_depth_to_color/camera_info</remapping>
-          <remapping>points:=depth/color/points</remapping>
+          <remapping>wrist_camera/image_raw:=color/image_raw</remapping>
+          <remapping>wrist_camera/camera_info:=color/camera_info</remapping>
+          <remapping>wrist_camera/depth/image_raw:=aligned_depth_to_color/image_raw</remapping>
+          <remapping>wrist_camera/depth/camera_info:=aligned_depth_to_color/camera_info</remapping>
+          <remapping>wrist_camera/points:=depth/color/points</remapping>
         </ros>
         <camera_name>wrist_camera</camera_name>
@@ -113,5 +117,8 @@
         <hack_baseline>0.018</hack_baseline>
         <min_depth>0.07</min_depth>
-        <max_depth>0.5</max_depth>
+        <!-- The look pose sees the cube at about 2 m from the spawn, and at
+             about 1.2 m once the base is beside the stand. 0.5 m returned
+             no range for either view. -->
+        <max_depth>3.0</max_depth>
       </plugin>
     </sensor>

File: src/steve_simulation/components/dynamixel/dynamixel_motor_xl-430.urdf.xacro (robot description, xacro)
@@ -45,5 +45,7 @@
         <origin xyz="0 0 0.0" rpy="${position_offset} 0 ${M_PI}"/>
         <axis xyz="${motor_direction} 0 0"/>
-        <limit effort="1.5" lower="-${M_PI / 180 * 180}" upper="${M_PI / 180 * 20}" velocity="6.178465545"/>
+        <!-- +20 deg cannot pitch the head down onto the cube. Full turn
+             matches the ros2_control command limits. -->
+        <limit effort="1.5" lower="-${M_PI}" upper="${M_PI}" velocity="6.178465545"/>
         <dynamics damping="0.7" friction="0.5"/>
       </joint>

File: src/steve_simulation/components/pan_tilt/pan_tilt.ros2_control.xacro (robot description, xacro)
@@ -23,5 +23,5 @@
         </command_interface>
         <state_interface name="position">
-          <param name="initial_value">-0.2</param>
+          <param name="initial_value">0.41</param>
         </state_interface>
         <state_interface name="velocity"/>
